File: Hardware/kicad_proj/ProIMU_V1/CAN_TRX.kicad_sch (KiCad schematic)
At the start: 6 parts

Commit message: Update: Schematic
Parts:
- added CAN?: Conn_02x02_Counter_Clockwise, symbol Connector_Generic:Conn_02x02_Counter_Clockwise
Connections:
- net GND: now also CAN?.2 (Pin_2)
- net CAN_RXD: no longer names the net of U?.4 (RXD)
- net CAN_RXD: now also CAN?.4 (Pin_4)
- net CAN_TXD: no longer names the net of U?.1 (TXD)
- net CAN_TXD: now also CAN?.3 (Pin_3)
- new net VDD: CAN?.1 (Pin_1)
Other:
- moved on the sheet: C?
Changed lines of the file:
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@@
   (junction (at 170.18 78.74) (diameter 0) (color 0 0 0 0)
   )
-  (junction (at 127 62.23) (diameter 0) (color 0 0 0 0)
-  )
-  (wire (pts (xy 123.19 83.82) (xy 133.35 83.82))
-    (stroke (width 0) (type default) (color 0 0 0 0))
+  (junction (at 105.41 62.23) (diameter 0) (color 0 0 0 0)
   )
   (wire (pts (xy 162.56 100.33) (xy 170.18 100.33))
     (stroke (width 0) (type default) (color 0 0 0 0))
   )
-  (wire (pts (xy 121.92 64.77) (xy 121.92 62.23))
+  (wire (pts (xy 100.33 64.77) (xy 100.33 62.23))
     (stroke (width 0) (type default) (color 0 0 0 0))
   )
@@
     (stroke (width 0) (type default) (color 0 0 0 0))
   )
-  (wire (pts (xy 121.92 62.23) (xy 127 62.23))
+  (wire (pts (xy 100.33 62.23) (xy 105.41 62.23))
     (stroke (width 0) (type default) (color 0 0 0 0))
   )
@@
     (stroke (width 0) (type default) (color 0 0 0 0))
   )
+  (wire (pts (xy 82.55 91.44) (xy 82.55 83.82))
+    (stroke (width 0) (type default) (color 0 0 0 0))
+  )
   (wire (pts (xy 149.86 116.84) (xy 149.86 119.38))
     (stroke (width 0) (type default) (color 0 0 0 0))
   )
-  (wire (pts (xy 121.92 69.85) (xy 121.92 72.39))
-    (stroke (width 0) (type default) (color 0 0 0 0))
-  )
-  (wire (pts (xy 127 86.36) (xy 127 62.23))
+  (wire (pts (xy 100.33 69.85) (xy 100.33 72.39))
+    (stroke (width 0) (type default) (color 0 0 0 0))
+  )
+  (wire (pts (xy 105.41 86.36) (xy 105.41 62.23))
     (stroke (width 0) (type default) (color 0 0 0 0))
   )
@@
     (stroke (width 0) (type default) (color 0 0 0 0))
   )
+  (wire (pts (xy 87.63 93.98) (xy 82.55 93.98))
+    (stroke (width 0) (type default) (color 0 0 0 0))
+  )
   (wire (pts (xy 162.56 91.44) (xy 162.56 100.33))
     (stroke (width 0) (type default) (color 0 0 0 0))
@@
     (stroke (width 0) (type default) (color 0 0 0 0))
   )
-  (wire (pts (xy 120.65 93.98) (xy 133.35 93.98))
+  (wire (pts (xy 82.55 93.98) (xy 82.55 97.79))
+    (stroke (width 0) (type default) (color 0 0 0 0))
+  )
+  (wire (pts (xy 100.33 93.98) (xy 133.35 93.98))
     (stroke (width 0) (type default) (color 0 0 0 0))
   )
@@
     (stroke (width 0) (type default) (color 0 0 0 0))
   )
-  (wire (pts (xy 120.65 91.44) (xy 133.35 91.44))
+  (wire (pts (xy 100.33 91.44) (xy 133.35 91.44))
     (stroke (width 0) (type default) (color 0 0 0 0))
   )
@@
     (stroke (width 0) (type default) (color 0 0 0 0))
   )
-  (wire (pts (xy 133.35 86.36) (xy 127 86.36))
+  (wire (pts (xy 133.35 86.36) (xy 105.41 86.36))
+    (stroke (width 0) (type default) (color 0 0 0 0))
+  )
+  (wire (pts (xy 87.63 91.44) (xy 82.55 91.44))
     (stroke (width 0) (type default) (color 0 0 0 0))
   )
@@
     (stroke (width 0) (type default) (color 0 0 0 0))
   )
-  (wire (pts (xy 127 62.23) (xy 127 60.96))
+  (wire (pts (xy 105.41 62.23) (xy 105.41 60.96))
+    (stroke (width 0) (type default) (color 0 0 0 0))
+  )
+  (wire (pts (xy 124.46 83.82) (xy 133.35 83.82))
     (stroke (width 0) (type default) (color 0 0 0 0))
   )
@@
     (stroke (width 0) (type default) (color 0 0 0 0))
   )
-  (hierarchical_label "CAN_TXD" (shape input) (at 120.65 93.98 180)
+  (global_label "CAN_H" (shape input) (at 195.58 100.33 0) (fields_autoplaced)
+    (effects (font (size 1.27 1.27)) (justify left))
+    (property "Intersheet References" "${INTERSHEET_REFS}" (id 0) (at 203.9802 100.2506 0)
+      (effects (font (size 1.27 1.27)) (justify left) hide)
+    )
+  )
+  (global_label "CAN_SHUTDOWN" (shape input) (at 124.46 83.82 180) (fields_autoplaced)
     (effects (font (size 1.27 1.27)) (justify right))
-  )
-  (hierarchical_label "CAN_L" (shape input) (at 195.58 78.74 0)
+    (property "Intersheet References" "${INTERSHEET_REFS}" (id 0) (at 107.1698 83.7406 0)
+      (effects (font (size 1.27 1.27)) (justify right) hide)
+    )
+  )
+  (global_label "CAN_L" (shape input) (at 195.58 78.74 0) (fields_autoplaced)
     (effects (font (size 1.27 1.27)) (justify left))
-  )
-  (hierarchical_label "CAN_H" (shape input) (at 195.58 100.33 0)
-    (effects (font (size 1.27 1.27)) (justify left))
-  )
-  (hierarchical_label "CAN_SHUTDOWN" (shape input) (at 123.19 83.82 180)
-    (effects (font (size 1.27 1.27)) (justify right))
-  )
-  (hierarchical_label "CAN_RXD" (shape input) (at 120.65 91.44 180)
-    (effects (font (size 1.27 1.27)) (justify right))
+    (property "Intersheet References" "${INTERSHEET_REFS}" (id 0) (at 203.6779 78.6606 0)
+      (effects (font (size 1.27 1.27)) (justify left) hide)
+    )
   )
   (symbol (lib_id "Device:R_Small") (at 170.18 93.98 0) (unit 1)
@@
     (pin "2")
   )
-  (symbol (lib_id "power:GND") (at 121.92 72.39 0) (mirror y) (unit 1)
-    (in_bom yes) (on_board yes)
-    (property "Reference" "#PWR?" (id 0) (at 121.92 78.74 0)
-      (effects (font (size 1.27 1.27)) hide)
-    )
-    (property "Value" "GND" (id 1) (at 119.38 76.2 0)
-      (effects (font (size 1.27 1.27)) (justify right))
-    )
-    (property "Footprint" "" (id 2) (at 121.92 72.39 0)
-      (effects (font (size 1.27 1.27)) hide)
-    )
-    (property "Datasheet" "" (id 3) (at 121.92 72.39 0)
+  (symbol (lib_id "power:VDD") (at 82.55 83.82 0) (unit 1)
+    (in_bom yes) (on_board yes) (fields_autoplaced)
+    (property "Reference" "#PWR?" (id 0) (at 82.55 87.63 0)
+      (effects (font (size 1.27 1.27)) hide)
+    )
+    (property "Value" "VDD" (id 1) (at 82.55 78.74 0))
+    (property "Footprint" "" (id 2) (at 82.55 83.82 0)
+      (effects (font (size 1.27 1.27)) hide)
+    )
+    (property "Datasheet" "" (id 3) (at 82.55 83.82 0)
+      (effects (font (size 1.27 1.27)) hide)
+    )
+    (pin "1")
+  )
+  (symbol (lib_id "power:GND") (at 100.33 72.39 0) (mirror y) (unit 1)
+    (in_bom yes) (on_board yes)
+    (property "Reference" "#PWR?" (id 0) (at 100.33 78.74 0)
+      (effects (font (size 1.27 1.27)) hide)
+    )
+    (property "Value" "GND" (id 1) (at 97.79 76.2 0)
+      (effects (font (size 1.27 1.27)) (justify right))
+    )
+    (property "Footprint" "" (id 2) (at 100.33 72.39 0)
+      (effects (font (size 1.27 1.27)) hide)
+    )
+    (property "Datasheet" "" (id 3) (at 100.33 72.39 0)
       (effects (font (size 1.27 1.27)) hide)
     )
@@
     (pin "1")
     (pin "2")
+  )
+  (symbol (lib_id "power:GND") (at 82.55 97.79 0) (unit 1)
+    (in_bom yes) (on_board yes) (fields_autoplaced)
+    (property "Reference" "#PWR?" (id 0) (at 82.55 104.14 0)
+      (effects (font (size 1.27 1.27)) hide)
+    )
+    (property "Value" "GND" (id 1) (at 82.55 102.87 0))
+    (property "Footprint" "" (id 2) (at 82.55 97.79 0)
+      (effects (font (size 1.27 1.27)) hide)
+    )
+    (property "Datasheet" "" (id 3) (at 82.55 97.79 0)
+      (effects (font (size 1.27 1.27)) hide)
+    )
+    (pin "1")
   )
   (symbol (lib_id "Interface_CAN_LIN:TJA1051T-3") (at 146.05 88.9 0) (mirror x) (unit 1)
@@
     (pin "8")
   )
-  (symbol (lib_id "Device:C_Small") (at 121.92 67.31 0) (mirror x) (unit 1)
-    (in_bom yes) (on_board yes) (fields_autoplaced)
-    (property "Reference" "C?" (id 0) (at 119.38 66.0335 0)
-      (effects (font (size 1.27 1.27)) (justify right))
-    )
-    (property "Value" "1uF" (id 1) (at 119.38 68.5735 0)
-      (effects (font (size 1.27 1.27)) (justify right))
-    )
-    (property "Footprint" "Capacitor_SMD:C_0402_1005Metric_Pad0.74x0.62mm_HandSolder" (id 2) (at 121.92 67.31 0)
-      (effects (font (size 1.27 1.27)) hide)
-    )
-    (property "Datasheet" "~" (id 3) (at 121.92 67.31 0)
-      (effects (font (size 1.27 1.27)) hide)
-    )
-    (pin "1")
-    (pin "2")
+  (symbol (lib_id "Device:C_Small") (at 100.33 67.31 0) (mirror x) (unit 1)
+    (in_bom yes) (on_board yes) (fields_autoplaced)
+    (property "Reference" "C?" (id 0) (at 97.79 66.0335 0)
+      (effects (font (size 1.27 1.27)) (justify right))
+    )
+    (property "Value" "1uF" (id 1) (at 97.79 68.5735 0)
+      (effects (font (size 1.27 1.27)) (justify right))
+    )
+    (property "Footprint" "Capacitor_SMD:C_0402_1005Metric_Pad0.74x0.62mm_HandSolder" (id 2) (at 100.33 67.31 0)
+      (effects (font (size 1.27 1.27)) hide)
+    )
+    (property "Datasheet" "~" (id 3) (at 100.33 67.31 0)
+      (effects (font (size 1.27 1.27)) hide)
+    )
+    (pin "1")
+    (pin "2")
+  )
+  (symbol (lib_id "Connector_Generic:Conn_02x02_Counter_Clockwise") (at 92.71 91.44 0) (unit 1)
+    (in_bom yes) (on_board yes)
+    (property "Reference" "CAN?" (id 0) (at 93.98 87.63 0))
+    (property "Value" "Conn_02x02_Counter_Clockwise" (id 1) (at 93.98 106.68 0))
+    (property "Footprint" "" (id 2) (at 92.71 91.44 0)
+      (effects (font (size 1.27 1.27)) hide)
+    )
+    (property "Datasheet" "~" (id 3) (at 92.71 91.44 0)
+      (effects (font (size 1.27 1.27)) hide)
+    )
+    (pin "1")
+    (pin "2")
+    (pin "3")
+    (pin "4")
   )
   (symbol (lib_id "power:+5V") (at 154.94 100.33 0) (mirror y) (unit 1)
@@
     (pin "1")
   )
-  (symbol (lib_id "power:+3V3") (at 127 60.96 0) (mirror y) (unit 1)
-    (in_bom yes) (on_board yes) (fields_autoplaced)
-    (property "Reference" "#PWR?" (id 0) (at 127 64.77 0)
-      (effects (font (size 1.27 1.27)) hide)
-    )
-    (property "Value" "+3V3" (id 1) (at 129.54 59.6899 0)
-      (effects (font (size 1.27 1.27)) (justify right))
-    )
-    (property "Footprint" "" (id 2) (at 127 60.96 0)
-      (effects (font (size 1.27 1.27)) hide)
-    )
-    (property "Datasheet" "" (id 3) (at 127 60.96 0)
-      (effects (font (size 1.27 1.27)) hide)
-    )
+  (symbol (lib_id "power:+3V3") (at 105.41 60.96 0) (mirror y) (unit 1)
+    (in_bom yes) (on_board yes) (fields_autoplaced)
+    (property "Reference" "#PWR?" (id 0) (at 105.41 64.77 0)
+      (effects (font (size 1.27 1.27)) hide)
+    )
+    (property "Value" "+3V3" (id 1) (at 107.95 59.6899 0)
+      (effects (font (size 1.27 1.27)) (justify right))
+    )
+    (property "Footprint" "" (id 2) (at 105.41 60.96 0)
+      (effects (font (size 1.27 1.27)) hide)
+    )
+    (property "Datasheet" "" (id 3) (at 105.41 60.96 0)
+      (effects (font (size 1.27 1.27)) hide)
+    )
