File: Hardware/kicad_proj/ProIMU_V1/RS485_Isolator.kicad_sch (KiCad schematic)
At the start: 1 part

Commit message: Update: Schematic
Parts:
- added RS?: Conn_02x03_Counter_Clockwise, symbol Connector_Generic:Conn_02x03_Counter_Clockwise
Connections:
- new net VDD: RS?.3 (Pin_3)
Changed lines of the file:
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@@
   (junction (at 124.46 78.74) (diameter 0) (color 0 0 0 0)
+  )
+  (wire (pts (xy 91.44 114.3) (xy 91.44 109.22))
+    (stroke (width 0) (type default) (color 0 0 0 0))
   )
   (wire (pts (xy 114.3 73.66) (xy 130.81 73.66))
@@
   )
   (wire (pts (xy 114.3 78.74) (xy 124.46 78.74))
+    (stroke (width 0) (type default) (color 0 0 0 0))
+  )
+  (wire (pts (xy 92.71 116.84) (xy 92.71 107.95))
+    (stroke (width 0) (type default) (color 0 0 0 0))
+  )
+  (wire (pts (xy 57.15 121.92) (xy 68.58 121.92))
     (stroke (width 0) (type default) (color 0 0 0 0))
   )
@@
   )
   (wire (pts (xy 161.29 73.66) (xy 182.88 73.66))
+    (stroke (width 0) (type default) (color 0 0 0 0))
+  )
+  (wire (pts (xy 81.28 124.46) (xy 106.68 124.46))
     (stroke (width 0) (type default) (color 0 0 0 0))
   )
@@
     (stroke (width 0) (type default) (color 0 0 0 0))
   )
+  (wire (pts (xy 92.71 107.95) (xy 57.15 107.95))
+    (stroke (width 0) (type default) (color 0 0 0 0))
+  )
   (wire (pts (xy 114.3 71.12) (xy 130.81 71.12))
     (stroke (width 0) (type default) (color 0 0 0 0))
@@
     (stroke (width 0) (type default) (color 0 0 0 0))
   )
+  (wire (pts (xy 81.28 119.38) (xy 106.68 119.38))
+    (stroke (width 0) (type default) (color 0 0 0 0))
+  )
+  (wire (pts (xy 58.42 109.22) (xy 91.44 109.22))
+    (stroke (width 0) (type default) (color 0 0 0 0))
+  )
+  (wire (pts (xy 58.42 119.38) (xy 68.58 119.38))
+    (stroke (width 0) (type default) (color 0 0 0 0))
+  )
+  (wire (pts (xy 58.42 124.46) (xy 68.58 124.46))
+    (stroke (width 0) (type default) (color 0 0 0 0))
+  )
   (wire (pts (xy 114.3 66.04) (xy 130.81 66.04))
+    (stroke (width 0) (type default) (color 0 0 0 0))
+  )
+  (wire (pts (xy 106.68 116.84) (xy 92.71 116.84))
+    (stroke (width 0) (type default) (color 0 0 0 0))
+  )
+  (wire (pts (xy 57.15 107.95) (xy 57.15 121.92))
+    (stroke (width 0) (type default) (color 0 0 0 0))
+  )
+  (wire (pts (xy 58.42 109.22) (xy 58.42 119.38))
+    (stroke (width 0) (type default) (color 0 0 0 0))
+  )
+  (wire (pts (xy 81.28 121.92) (xy 106.68 121.92))
+    (stroke (width 0) (type default) (color 0 0 0 0))
+  )
+  (wire (pts (xy 106.68 114.3) (xy 91.44 114.3))
     (stroke (width 0) (type default) (color 0 0 0 0))
   )
@@
   (hierarchical_label "RS485_TX+" (shape input) (at 114.3 66.04 180)
     (effects (font (size 1.27 1.27)) (justify right))
+  )
+  (symbol (lib_id "power:VDD") (at 58.42 124.46 90) (unit 1)
+    (in_bom yes) (on_board yes)
+    (property "Reference" "#PWR?" (id 0) (at 62.23 124.46 0)
+      (effects (font (size 1.27 1.27)) hide)
+    )
+    (property "Value" "VDD" (id 1) (at 54.61 124.46 90)
+      (effects (font (size 1.27 1.27)) (justify left))
+    )
+    (property "Footprint" "" (id 2) (at 58.42 124.46 0)
+      (effects (font (size 1.27 1.27)) hide)
+    )
+    (property "Datasheet" "" (id 3) (at 58.42 124.46 0)
+      (effects (font (size 1.27 1.27)) hide)
+    )
+    (pin "1")
   )
   (symbol (lib_id "Interface_UART:ADM2582E") (at 146.05 73.66 0) (mirror y) (unit 1)
@@
     (pin "9")
   )
+  (symbol (lib_id "Connector_Generic:Conn_02x03_Counter_Clockwise") (at 73.66 121.92 0) (unit 1)
+    (in_bom yes) (on_board yes) (fields_autoplaced)
+    (property "Reference" "RS?" (id 0) (at 74.93 113.03 0))
+    (property "Value" "Conn_02x03_Counter_Clockwise" (id 1) (at 74.93 115.57 0))
+    (property "Footprint" "" (id 2) (at 73.66 121.92 0)
+      (effects (font (size 1.27 1.27)) hide)
+    )
+    (property "Datasheet" "~" (id 3) (at 73.66 121.92 0)
+      (effects (font (size 1.27 1.27)) hide)
+    )
+    (pin "1")
+    (pin "2")
+    (pin "3")
+    (pin "4")
+    (pin "5")
+    (pin "6")
+  )
 )
