File: Hardware/kicad_proj/ProIMU_V1/BMP280.kicad_sch (KiCad schematic)
At the start: 5 parts

Commit message: Update: Schematic
Parts:
- removed C? (x2): 100nF, Capacitor_SMD:C_0402_1005Metric_Pad0.74x0.62mm_HandSolder, symbol Device:C_Small
- removed R? (x2): 2.2K, Resistor_SMD:R_0402_1005Metric_Pad0.72x0.64mm_HandSolder, symbol Device:R_Small
- removed U?: BMP280, footprints:BMP280, symbol 2022-02-05_19-44-07:BMP280
Other:
- note removed: "BMP280: Barometer and Temperature Sensor"
