File: Hardware/kicad_proj/ProIMU_V1/ProIMU_V1.kicad_pcb (KiCad board)
At the start: 2 copper layers, 50 x 50 mm, 50 parts, among them IC1 MP2731GQC-0000-Z, J4 502570-0893, U1 ADM2582E, U2 TJA1051T-3, U4 AIR602, U5 BMP280, U6 MPU-9250, U7 TPS54308, U8 TPS54308, U9 STM32F412CEU6

Commit message: Updated repo
Parts:
- removed RS485: 43045-0609, Connector_JST:JST_XH_S6B-XH-A-1_1x06_P2.50mm_Horizontal
- added C1: 1uF, Capacitor_SMD:C_0402_1005Metric_Pad0.74x0.62mm_HandSolder, B.Cu at (143.5, 106.1)
- added C21: 1uF, Capacitor_SMD:C_0402_1005Metric_Pad0.74x0.62mm_HandSolder, B.Cu at (135.8, 124.0)
- added C22: 1uF, Capacitor_SMD:C_0402_1005Metric_Pad0.74x0.62mm_HandSolder, B.Cu at (139.0, 128.0)
- added C4: 1uF, Capacitor_SMD:C_0402_1005Metric_Pad0.74x0.62mm_HandSolder, B.Cu at (141.5, 125.5)
- added J3: Conn_01x06, Connector_PinHeader_1.27mm:PinHeader_2x03_P1.27mm_Vertical_SMD, F.Cu at (127.0, 92.6)
- added RS232: Conn_01x04, Connector_JST:JST_PH_S4B-PH-SM4-TB_1x04-1MP_P2.00mm_Horizontal, F.Cu at (138.5, 125.0)
- BAT1, C17, C18, C20, C5, R1, R2, U2: moved to B.Cu
- CAN1: footprint Connector_JST:JST_PH_S4B-PH-K_1x04_P2.00mm_Horizontal -> Connector_JST:JST_PH_S4B-PH-SM4-TB_1x04-1MP_P2.00mm_Horizontal
- U1: value ADM2582E -> ADM101E; footprint Package_SO:SOIC-20W_7.5x12.8mm_P1.27mm -> Package_SO:MSOP-10_3x3mm_P0.5mm
- U5: moved to F.Cu
- moved C5 108.3 mm to (158.2, 126.5), turned to 90 degrees
- moved C18 98.0 mm to (153.3, 102.0), turned to -90 degrees
- moved C17 89.5 mm to (151.5, 109.9), turned to 180 degrees
- moved R11 88.9 mm to (147.8, 99.1), turned to -90 degrees
- moved R5 81.4 mm to (162.0, 105.5), turned to 90 degrees
- moved R1 81.3 mm to (157.0, 126.5), turned to 90 degrees
- moved R2 78.7 mm to (159.5, 126.5), turned to -90 degrees
- moved BAT1 62.5 mm to (161.3, 83.0), turned to -90 degrees
- moved R6 61.5 mm to (160.7, 105.5), turned to 90 degrees
- moved C19 56.0 mm to (190.0, 95.4)
- moved J4 54.6 mm to (200.6, 114.1), turned to 90 degrees
- moved U1 51.4 mm to (138.4, 124.1), turned to 90 degrees
- moved IC1 36.3 mm to (162.5, 88.5)
- moved U7 21.8 mm to (228.7, 16.4)
- moved CAN1 6.24 mm to (158.5, 124.8)
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Connections:
- net /MCU/RS485_DE renamed /MCU/RS232_TX
- net /MCU/RS485_RXD renamed /MCU/RS232_RX
- U1 pad 1: GND -> GND2
- U1 pad 10: GND -> Net-(RS232-Pad1)
- U1 pad 2: +3V3 -> Net-(C4-Pad1)
- U1 pad 3: GND -> Net-(C22-Pad2)
- U1 pad 5: /MCU/RS485_nRE -> Net-(RS232-Pad4)
- U1 pad 7: /MCU/RS485_TXD -> Net-(RS232-Pad3)
- U1 pad 8: +3V3 -> unconnected-(U1-Pad8)
- U1 pad 9: GND -> Net-(C4-Pad2)
Routing:
- net +3V3: track 0.00 -> 12.1 mm, vias 0 -> 4
- net GND: track 0.00 -> 9.24 mm, vias 0 -> 6
- net /MCU/SWCLK: track 0.00 -> 7.24 mm
- net /MCU/DEBUG_UART_RX: track 0.00 -> 6.46 mm
- net /MCU/SWDIO: track 0.00 -> 6.25 mm
- net /MCU/DEBUG_UART_TX: track 0.00 -> 4.99 mm
- net /MCU/BMP280_SCK: track 0.00 -> 3.44 mm, vias 0 -> 2
- net /MCU/MCU_RESET: track 0.00 -> 3.24 mm
- net Net-(R11-Pad2): track 0.00 -> 1.89 mm
- net /MCU/BMP280_SDA: track 0.00 -> 1.79 mm
