File: Hardware/kicad_proj/ProIMU_V1/CAN.kicad_sch (KiCad schematic)
At the start: 11 parts

Commit message: Updated Schematic and Layout
Parts:
- gave numbers to parts that had none: 11
Changed lines of the file:
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@@
   (symbol (lib_id "power:+3V3") (at 180.34 27.94 0) (unit 1)
     (in_bom yes) (on_board yes) (fields_autoplaced)
-    (property "Reference" "#PWR?" (id 0) (at 180.34 31.75 0)
+    (property "Reference" "#PWR0110" (id 0) (at 180.34 31.75 0)
       (effects (font (size 1.27 1.27)) hide)
     )
@@
   (symbol (lib_id "power:GND") (at 180.34 63.5 0) (unit 1)
     (in_bom yes) (on_board yes)
-    (property "Reference" "#PWR?" (id 0) (at 180.34 69.85 0)
+    (property "Reference" "#PWR0112" (id 0) (at 180.34 69.85 0)
       (effects (font (size 1.27 1.27)) hide)
     )
@@
   (symbol (lib_id "Connector_Generic:Conn_01x04") (at 67.31 50.8 0) (mirror y) (unit 1)
     (in_bom yes) (on_board yes) (fields_autoplaced)
-    (property "Reference" "CAN?" (id 0) (at 67.31 41.91 0))
+    (property "Reference" "CAN1" (id 0) (at 67.31 41.91 0))
     (property "Value" "Conn_01x04" (id 1) (at 67.31 44.45 0))
     (property "Footprint" "Connector_JST:JST_PH_S4B-PH-SM4-TB_1x04-1MP_P2.00mm_Horizontal" (id 2) (at 67.31 50.8 0)
@@
   (symbol (lib_id "Device:R_Small") (at 85.09 78.74 0) (mirror x) (unit 1)
     (in_bom yes) (on_board yes)
-    (property "Reference" "R?" (id 0) (at 82.55 80.01 90)
+    (property "Reference" "R7" (id 0) (at 82.55 80.01 90)
       (effects (font (size 1.27 1.27)) (justify right))
     )
@@
   (symbol (lib_id "power:GND1") (at 153.67 63.5 0) (unit 1)
     (in_bom yes) (on_board yes)
-    (property "Reference" "#PWR?" (id 0) (at 153.67 69.85 0)
+    (property "Reference" "#PWR0113" (id 0) (at 153.67 69.85 0)
       (effects (font (size 1.27 1.27)) hide)
     )
@@
   (symbol (lib_id "Simulation_SPICE:DIODE") (at 88.9 31.75 0) (unit 1)
     (in_bom yes) (on_board yes) (fields_autoplaced)
-    (property "Reference" "D?" (id 0) (at 88.9 25.4 0))
+    (property "Reference" "D3" (id 0) (at 88.9 25.4 0))
     (property "Value" "DIODE" (id 1) (at 88.9 27.94 0))
     (property "Footprint" "" (id 2) (at 88.9 31.75 0)
@@
   (symbol (lib_id "Device:C_Small") (at 185.42 33.02 0) (mirror x) (unit 1)
     (in_bom yes) (on_board yes)
-    (property "Reference" "C?" (id 0) (at 189.23 31.75 0)
+    (property "Reference" "C5" (id 0) (at 189.23 31.75 0)
       (effects (font (size 1.27 1.27)) (justify right))
     )
@@
   (symbol (lib_id "Device:C_Small") (at 120.65 67.31 0) (mirror x) (unit 1)
     (in_bom yes) (on_board yes)
-    (property "Reference" "C?" (id 0) (at 119.38 66.04 90)
+    (property "Reference" "C4" (id 0) (at 119.38 66.04 90)
       (effects (font (size 1.27 1.27)) (justify right))
     )
@@
   (symbol (lib_id "Device:R_Small") (at 95.25 60.96 90) (mirror x) (unit 1)
     (in_bom yes) (on_board yes)
-    (property "Reference" "R?" (id 0) (at 93.98 60.96 90)
+    (property "Reference" "R9" (id 0) (at 93.98 60.96 90)
       (effects (font (size 1.27 1.27)) (justify right))
     )
@@
   (symbol (lib_id "Interface_CAN_LIN:ISO1050DUB") (at 165.1 50.8 0) (mirror y) (unit 1)
     (in_bom yes) (on_board yes) (fields_autoplaced)
-    (property "Reference" "U?" (id 0) (at 165.1 40.64 0))
+    (property "Reference" "U1" (id 0) (at 165.1 40.64 0))
     (property "Value" "ISO1050DUB" (id 1) (at 165.1 43.18 0))
     (property "Footprint" "Package_SO:SOP-8_6.62x9.15mm_P2.54mm" (id 2) (at 165.1 59.69 0)
@@
   (symbol (lib_id "Device:R_Small") (at 85.09 71.12 0) (mirror x) (unit 1)
     (in_bom yes) (on_board yes)
-    (property "Reference" "R?" (id 0) (at 82.55 72.39 90)
+    (property "Reference" "R6" (id 0) (at 82.55 72.39 90)
       (effects (font (size 1.27 1.27)) (justify right))
     )
@@
   (symbol (lib_id "power:GND1") (at 74.93 63.5 0) (unit 1)
     (in_bom yes) (on_board yes)
-    (property "Reference" "#PWR?" (id 0) (at 74.93 69.85 0)
+    (property "Reference" "#PWR0114" (id 0) (at 74.93 69.85 0)
       (effects (font (size 1.27 1.27)) hide)
     )
@@
   (symbol (lib_id "power:VDD") (at 123.19 24.13 0) (unit 1)
     (in_bom yes) (on_board yes) (fields_autoplaced)
-    (property "Reference" "#PWR?" (id 0) (at 123.19 27.94 0)
+    (property "Reference" "#PWR0109" (id 0) (at 123.19 27.94 0)
       (effects (font (size 1.27 1.27)) hide)
     )
@@
   (symbol (lib_id "power:GND") (at 185.42 38.1 0) (unit 1)
     (in_bom yes) (on_board yes)
-    (property "Reference" "#PWR?" (id 0) (at 185.42 44.45 0)
+    (property "Reference" "#PWR0111" (id 0) (at 185.42 44.45 0)
       (effects (font (size 1.27 1.27)) hide)
     )
@@
   (symbol (lib_id "Device:R_Small") (at 95.25 43.18 90) (mirror x) (unit 1)
     (in_bom yes) (on_board yes)
-    (property "Reference" "R?" (id 0) (at 93.98 43.18 90)
+    (property "Reference" "R8" (id 0) (at 93.98 43.18 90)
       (effects (font (size 1.27 1.27)) (justify right))
     )
@@
   (symbol (lib_id "power:GND1") (at 120.65 72.39 0) (unit 1)
     (in_bom yes) (on_board yes)
-    (property "Reference" "#PWR?" (id 0) (at 120.65 78.74 0)
+    (property "Reference" "#PWR0116" (id 0) (at 120.65 78.74 0)
       (effects (font (size 1.27 1.27)) hide)
     )
@@
   (symbol (lib_id "power:GND") (at 85.09 92.71 0) (unit 1)
     (in_bom yes) (on_board yes) (fields_autoplaced)
-    (property "Reference" "#PWR?" (id 0) (at 85.09 99.06 0)
+    (property "Reference" "#PWR0115" (id 0) (at 85.09 99.06 0)
       (effects (font (size 1.27 1.27)) hide)
     )
@@
   (symbol (lib_id "Device:R_Small") (at 128.27 55.88 0) (mirror y) (unit 1)
     (in_bom yes) (on_board yes)
-    (property "Reference" "R?" (id 0) (at 129.54 57.15 0)
+    (property "Reference" "R12" (id 0) (at 129.54 57.15 0)
       (effects (font (size 1.27 1.27)) (justify right))
     )
@@
   (symbol (lib_id "Device:R_Small") (at 128.27 48.26 0) (mirror y) (unit 1)
     (in_bom yes) (on_board yes)
-    (property "Reference" "R?" (id 0) (at 129.54 49.53 0)
-      (effects (font (size 1.27 1.27)) (justify right))
-    )
+    (property "Reference" "R10" (id 0) (at 129.54 49.53 0)
+      (effects (font (size 1.27 1.27)) (justify right))
+    )

Commit message: Updated Repo
Parts:
- added U11: SN65HVD235, Package_SO:SOIC-8_3.9x4.9mm_P1.27mm, symbol Interface_CAN_LIN:SN65HVD235
Changed lines of the file:
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@@
     (pin "2")
+  )
+  (symbol (lib_id "Interface_CAN_LIN:SN65HVD235") (at 163.83 87.63 0) (unit 1)
+    (in_bom yes) (on_board yes) (fields_autoplaced)
+    (property "Reference" "U11" (id 0) (at 165.8494 77.47 0)
+      (effects (font (size 1.27 1.27)) (justify left))
+    )
+    (property "Value" "SN65HVD235" (id 1) (at 165.8494 80.01 0)
+      (effects (font (size 1.27 1.27)) (justify left))
+    )
+    (property "Footprint" "Package_SO:SOIC-8_3.9x4.9mm_P1.27mm" (id 2) (at 163.83 100.33 0)
+      (effects (font (size 1.27 1.27)) hide)
+    )
+    (property "Datasheet" "http://www.ti.com/lit/ds/symlink/sn65hvd234.pdf" (id 3) (at 161.29 77.47 0)
+      (effects (font (size 1.27 1.27)) hide)
+    )
+    (pin "1")
+    (pin "2")
+    (pin "3")
+    (pin "4")
+    (pin "5")
+    (pin "6")
+    (pin "7")
+    (pin "8")
   )
   (symbol (lib_id "Device:R_Small") (at 128.27 48.26 0) (mirror y) (unit 1)
